Commit message: removed extra link causing gap between EE and last arm link

File: polymetis/polymetis/data/franka_panda_robotiq_85/panda_robotiq_85.urdf (robot description, URDF)
Before this commit: robot panda, 22 links, 21 joints
Links:
- removed link panda_link8
Joints:
- removed joint panda_joint8
- joint panda_joint_ee: parent panda_link8 -> panda_link7
